File: PCB/Audio Synthesizer.kicad_pcb (KiCad board)
At the start: 2 copper layers, 190 x 83.8 mm, 42 parts, among them J1 Conn_01x20, J2 Conn_01x05, J3 Conn_01x02, J4 Conn_01x20, SW1 SW_Push, SW10 SW_Push, SW11 SW_Push, SW12 SW_Push, SW13 SW_Push, SW14 SW_Push, SW15 SW_Push, SW16 SW_Push, SW17 RotaryEncoder_Switch, SW18 RotaryEncoder_Switch, SW2 SW_Push, SW3 SW_Push, SW4 SW_Push, SW5 SW_Push, SW6 SW_Push, SW7 SW_Push, SW8 SW_Push, SW9 SW_Push

Commit message: Add files via upload
Parts:
- removed RV1: R_Potentiometer_Trim, Potentiometer_THT:Potentiometer_Bourns_PTA2043_Single_Slide
Routing:
- net /GPIO26: track 109.6 -> 0.00 mm
- net +3V3: track 122.2 -> 57.7 mm, vias 3 -> 1
